Commit message: add motor link

File: hexar_description/urdf/hexar.urdf (robot description, URDF)
Before this commit: robot hexar, 3 links, 2 joints
Links:
- added link left_motor, mass 0.101; collision cylinder length=0.067 radius=0.0125; visual cylinder length=0.067 radius=0.0125
- added link right_bracket, mass 0.0085; collision box size=0.025 0.052 0.002; visual box size=0.025 -0.052 0.002
- link caster_wheel: mass 0.004 -> 0.0165
- link left_bracket: mass 0.004 -> 0.0085
Joints:
- added joint chassis-right_bracket: type fixed, parent chassis, child right_bracket, origin xyz=-0.0375 0.061 -0.0005 rpy=0 0 0
- added joint left_bracket-left_motor: type fixed, parent left_bracket, child left_motor, origin xyz=0 -0.0075 0.0135 rpy=1.5707963267948966 0 0
- joint chassis-caster_wheel: origin xyz=0.0802 0 -0.0135 rpy=0 0 0 -> xyz=0.0802 0 -0.0143 rpy=0 0 0

Commit message: add wheels to urdf

File: hexar_description/urdf/hexar.urdf (robot description, URDF)
Before this commit: robot hexar, 5 links, 4 joints
Links:
- added link left_wheel, mass 0.023; collision cylinder length=0.01 radius=0.04; visual cylinder length=0.01 radius=0.04
- added link right_motor, mass 0.101; collision cylinder length=0.067 radius=0.0125; visual cylinder length=0.067 radius=0.0125
- added link right_wheel, mass 0.023; collision cylinder length=0.01 radius=0.04; visual cylinder length=0.01 radius=0.04
Joints:
- added joint left_motor-left_wheel: type continuous, parent left_motor, child left_wheel, origin xyz=0 -0 -0.045 rpy=0 0 0, axis 0 0 1
- added joint right_bracket-right_motor: type fixed, parent right_bracket, child right_motor, origin xyz=0 0.0075 0.0135 rpy=1.5707963267948966 0 0
- added joint right_motor-right_wheel: type continuous, parent right_motor, child right_wheel, origin xyz=0 0 0.045 rpy=0 0 0, axis 0 0 1
- joint chassis-right_bracket: origin xyz=-0.0375 0.061 -0.0005 rpy=0 0 0 -> xyz=-0.0375 -0.061 -0.0005 rpy=0 0 0

Commit message: fix diff drive direction

File: hexar_description/urdf/hexar.urdf (robot description, URDF)
Before this commit: robot hexar, 8 links, 7 joints
Joints:
- joint left_bracket-left_motor: origin xyz=0 -0.0075 0.0135 rpy=1.5707963267948966 0 0 -> xyz=0 -0.0075 0.0135 rpy=-1.5707963267948966 0 0
- joint left_motor-left_wheel: origin xyz=0 -0 -0.045 rpy=0 0 0 -> xyz=0 -0 0.045 rpy=0 0 0
- joint right_bracket-right_motor: origin xyz=0 0.0075 0.0135 rpy=1.5707963267948966 0 0 -> xyz=0 0.0075 0.0135 rpy=-1.5707963267948966 0 0
- joint right_motor-right_wheel: origin xyz=0 0 0.045 rpy=0 0 0 -> xyz=0 0 -0.045 rpy=0 0 0

Commit message: add reduce size rplidar meshes

File: hexar_description/urdf/hexar.urdf (robot description, URDF)
Before this commit: robot hexar, 8 links, 7 joints
Links:
- added link lidar, mass 0.17; collision box size=0.1 0.055 0.07; visual mesh filename=package://hexar_description/meshes/rplidar_a1m8.dae
- link right_bracket: geometry collision box size=0.025 0.052 0.002; visual box size=0.025 0.052 0.002
Joints:
- added joint chassis-lidar: type fixed, parent chassis, child lidar, origin xyz=-0.025 0.038 0.0045 rpy=1.5707963267948966 0 0

Commit message: add laser sensor plugin

File: hexar_description/urdf/hexar.urdf (robot description, URDF)
Before this commit: robot hexar, 9 links, 8 joints
Links:
- removed link lidar
- added link laser_house, mass 0.17; collision box size=0.1 0.055 0.07; visual mesh filename=package://hexar_description/meshes/rplidar_a1m8.dae
- added link sensor
Joints:
- removed joint chassis-lidar
- added joint chassis-laser_house: type fixed, parent chassis, child laser_house, origin xyz=-0.025 0.038 0.0045 rpy=1.5707963267948966 0 0
- added joint chassis-sensor: type fixed, parent chassis, child sensor, origin xyz=0.013 0 0.042 rpy=0 0 0

Commit message: add inertia to chassis

File: hexar_description/urdf/hexar.urdf (robot description, URDF)
Before this commit: robot hexar, 10 links, 9 joints
Links:
- link chassis: mass None -> 0.1

Commit message: add footprint and rename chassis to base_link

File: hexar_description/urdf/hexar.urdf (robot description, URDF)
Before this commit: robot hexar, 10 links, 9 joints
Links:
- removed link chassis
- added link base_footprint
- added link base_inertial, mass 0.1
- added link base_link; collision cylinder length=0.009 radius=0.1; visual cylinder length=0.009 radius=0.1
Joints:
- removed joint chassis-caster_wheel
- removed joint chassis-laser_house
- removed joint chassis-left_bracket
- removed joint chassis-right_bracket
- removed joint chassis-sensor
- added joint base_link-base_footprint: type fixed, parent base_link, child base_footprint, origin xyz=0 0 -0.027 rpy=0 0 0
- added joint base_link-base_inertial: type fixed, parent base_link, child base_inertial, origin xyz=0 0 0 rpy=0 0 0
- added joint base_link-caster_wheel: type fixed, parent base_link, child caster_wheel, origin xyz=0.0802 0 -0.0143 rpy=0 0 0
- added joint base_link-laser_house: type fixed, parent base_link, child laser_house, origin xyz=-0.025 0.038 0.0045 rpy=1.5707963267948966 0 0
- added joint base_link-left_bracket: type fixed, parent base_link, child left_bracket, origin xyz=-0.0375 0.061 -0.0005 rpy=0 0 0
- added joint base_link-right_bracket: type fixed, parent base_link, child right_bracket, origin xyz=-0.0375 -0.061 -0.0005 rpy=0 0 0
- added joint base_link-sensor: type fixed, parent base_link, child sensor, origin xyz=0.013 0 0.042 rpy=0 0 0

Commit message: fix lidar urdf

File: hexar_description/urdf/hexar.urdf (robot description, URDF)
Before this commit: robot hexar, 12 links, 11 joints
Links:
- removed link caster_wheel
- removed link laser_house
- removed link sensor
- added link caster_ball, mass 0.0165; collision sphere radius=0.0127; visual sphere radius=0.0127
- added link lidar_house, mass 0.17; collision box size=0.1 0.055 0.07; visual mesh filename=package://hexar_description/meshes/rplidar_a1m8.dae
- added link lidar_sensor
Joints:
- removed joint base_link-caster_wheel
- removed joint base_link-laser_house
- removed joint base_link-sensor
- added joint base_link-caster_ball: type fixed, parent base_link, child caster_ball, origin xyz=0.0802 0 -0.0143 rpy=0 0 0
- added joint base_link-lidar_house: type fixed, parent base_link, child lidar_house, origin xyz=-0.025 0.038 0.0045 rpy=1.5707963267948966 0 0
- added joint base_link-lidar_sensor: type fixed, parent base_link, child lidar_sensor, origin xyz=0.013 0 0.042 rpy=0 0 0

Commit message: fix lidar, need manually set Reliability Policy to Best Effort to view laser scan points

File: hexar_description/urdf/hexar.urdf (robot description, URDF)
Before this commit: robot hexar, 12 links, 11 joints
Links:
- link lidar_house: geometry collision box size=0.1 0.055 0.07; visual mesh filename=file://$(find hexar_description)/meshes/rplidar_a1m8.dae
